Commit message: Update

File: description/robot_core.xacro (robot description, xacro)
@@ -42,5 +42,13 @@
     </link>
     <gazebo reference="chassis">
-        <material>Gazebo/White</material>
+        <visual>
+            <material>
+                <!-- Values between 0.0 and 1.0 -->
+                <ambient>1.0 1.0 1.0 1.0</ambient>
+                <diffuse>1.0 1.0 1.0 1.0</diffuse>
+                <specular>0.0 0.0 0.0 1.0</specular>
+                <emissive>0.0 0.0 0.0 1.0</emissive>
+            </material>
+        </visual>
     </gazebo>
     <!-- LEFT WHEEL LINK -->
@@ -69,5 +77,13 @@
     </link>
     <gazebo reference="left_wheel">
-        <material>Gazebo/Blue</material>
+        <visual>
+            <material>
+                <!-- Values between 0.0 and 1.0 -->
+                <ambient>0.0 0.0 1.0 1.0</ambient>
+                <diffuse>0.0 0.0 1.0 1.0</diffuse>
+                <specular>0.0 0.0 0.0 1.0</specular>
+                <emissive>0.0 0.0 0.0 1.0</emissive>
+            </material>
+        </visual>
     </gazebo>
     <!-- RIGHT WHEEL LINK -->
@@ -93,7 +109,15 @@
         </xacro:inertial_cylinder>
     </link>
-    <ignition reference="right_wheel">
-        <material> Gazebo/Red</material>
-    </ignition>
+    <gazebo reference="right_wheel">
+        <visual>
+            <material>
+                <!-- Values between 0.0 and 1.0 -->
+                <ambient>0.0 0.0 1.0 1.0</ambient>
+                <diffuse>0.0 0.0 1.0 1.0</diffuse>
+                <specular>0.0 0.0 0.0 1.0</specular>
+                <emissive>0.0 0.0 0.0 1.0</emissive>
+            </material>
+        </visual>
+    </gazebo>
     <!-- CASTER WHEEL LINK -->
     <joint name="caster_wheel_joint" type="continuous">
@@ -107,4 +131,5 @@
                 <sphere radius="0.05"/>
             </geometry>
+            <material name="black"/>
         </visual>
         <collision>
@@ -118,5 +143,13 @@
     </link>
     <gazebo reference="caster_wheel">
-        <material> Gazebo/Black</material>
+        <visual>
+            <material>
+                <!-- Values between 0.0 and 1.0 -->
+                <ambient>0.0 0.0 0.0 1.0</ambient>
+                <diffuse>0.0 0.0 0.0 1.0</diffuse>
+                <specular>0.0 0.0 0.0 1.0</specular>
+                <emissive>0.0 0.0 0.0 1.0</emissive>
+            </material>
+        </visual>
         <collision>
             <surface>
